File: power.sch (KiCad schematic (older format))
At the start: 0 parts

Commit message: Schematics: Power supply from battery input
Parts:
- added C? (x2): 10u, symbol C_Small
- added C?: 100n, symbol C_Small
- added C?: 10p, symbol C_Small
- added C? (x3): 22u, symbol C_Small
- added CONN?: PWR, MODULE, symbol PWR
- added D?: POWER, symbol Led_Small
- added L?: 1uH, symbol INDUCTOR_SMALL
- added Q?: Q_NMOS_DGS, symbol Q_NMOS_DGS
- added R? (x2): 1M, symbol R_Small
- added R?: 111k, symbol R_Small
- added R?: 1k, symbol R_Small
- added U?: TPS63060, symbol TPS63060
Connections:
- new net: L?.1, U?.1 (L1)
- new net: L?.2, U?.10 (L2)
- new net: C?.1, U?.6 (VAUX)
- new net: C?.1, R?.1, R?.2, U?.8 (FB)
- new net: Q?.3 (S), R?.1
- new net: D?.1 (K), Q?.1 (D)
- new net +5V: C?.1, C?.1, C?.1, D?.2 (A), R?.1, R?.1, U?.9 (VOUT)
- new net GND: C?.2, C?.2, C?.2, C?.2, C?.2, C?.2, C?.2, CONN?.2 (-), CONN?.MECH (GND), R?.2, R?.2, U?.11 (PGND), U?.4 (PS/SYNC), U?.7 (GND)
- new net POWER: C?.1, C?.1, CONN?.1 (+), U?.2 (VIN), U?.3 (EN)
- new net PWR_GOOD: Q?.2 (G), R?.2, U?.5 (PG)
Other:
- note added: "5V, 800mA output\nCan go up to 2A"
- note added: "If using TPS63061:\nReplace 1M by 0R\nand DNP 111k/10p"
- note added: "PWR_GOOD is\n1 if good (LED ON)\n0 if failure (LED OFF)"

Commit message: Schematics: GPS, Backup battery & Load Switch
Parts:
- added BT?: 1.4V to 3.6V, symbol Battery
- added C? (x2): 1u, symbol C_Small
- added F?: 500mA, symbol F_Small
- added U?: TPS22929D, symbol TPS22929D
Connections:
- net GND: now also BT?.2, C?.2, C?.2, U?.2 (GND), U?.5 (GND)
- new net: C?.1, F?.2, U?.4 (VIN), U?.6 (VIN)
- new net +3.3V_A: C?.1, U?.1 (VOUT)
- new net +3V3: F?.1
- new net 3.3V_A_EN: U?.3 (ON)
- new net Back_Bat: BT?.1
Changed lines of the file:
@@
 	2000 1550 2100 1550
 Wire Wire Line
-	5275 1600 6725 1600
+	5275 1600 5800 1600
+Wire Wire Line
+	5800 1600 6375 1600
+Wire Wire Line
+	6375 1600 6550 1600
+Wire Wire Line
+	6550 1600 6725 1600
 Connection ~ 5800 1600
 Wire Wire Line
@@
 	4125 2300 4125 2100
 Wire Wire Line
-	3550 2300 4175 2300
+	3550 2300 3725 2300
+Wire Wire Line
+	3725 2300 3900 2300
+Wire Wire Line
+	3900 2300 4125 2300
+Wire Wire Line
+	4125 2300 4175 2300
 Wire Wire Line
 	4125 2100 4175 2100
@@
 	3900 1900 4175 1900
 Wire Wire Line
-	3425 1600 4175 1600
+	3425 1600 3550 1600
+Wire Wire Line
+	3550 1600 3725 1600
+Wire Wire Line
+	3725 1600 4125 1600
+Wire Wire Line
+	4125 1600 4175 1600
 Wire Wire Line
 	3725 1600 3725 1650
@@
 Connection ~ 3550 1600
 Wire Wire Line
-	3550 1850 3550 2350
+	3550 1850 3550 2300
+Wire Wire Line
+	3550 2300 3550 2350
 Connection ~ 3550 2300
 Wire Wire Line
@@
 	5325 2300 5325 2350
 Wire Wire Line
-	5275 1800 6100 1800
+	5275 1800 5800 1800
+Wire Wire Line
+	5800 1800 6100 1800
 Connection ~ 5800 1800
 $Comp
@@
 	8425 1550 8425 1600
 Wire Wire Line
-	7975 1800 8125 1800
+	7975 1800 8075 1800
+Wire Wire Line
+	8075 1800 8125 1800
 $Comp
 L R_Small R?
@@
 $EndComp
 Wire Wire Line
-	8425 1300 8425 1350
+	8425 1300 8425 1325
+Wire Wire Line
+	8425 1325 8425 1350
 Wire Wire Line
 	8425 1325 8075 1325
@@
 $EndComp
 Wire Wire Line
-	6725 1550 6725 1675
+	6725 1550 6725 1600
+Wire Wire Line
+	6725 1600 6725 1675
 Connection ~ 6725 1600
 Wire Wire Line
@@
 $EndComp
 Wire Wire Line
-	5800 2025 6725 2025
-Wire Wire Line
-	6725 1875 6725 2050
+	5800 2025 6100 2025
+Wire Wire Line
+	6100 2025 6375 2025
+Wire Wire Line
+	6375 2025 6550 2025
+Wire Wire Line
+	6550 2025 6725 2025
+Wire Wire Line
+	6725 1875 6725 2025
+Wire Wire Line
+	6725 2025 6725 2050
 Connection ~ 6725 2025
 Wire Wire Line
@@
 	4125 1700 4125 1600
 Connection ~ 4125 1600
+$Comp
+L TPS22929D U?
+U 1 1 55AC0F91
+P 2600 3800
+F 0 "U?" H 2800 3350 60  0000 C CNN
+F 1 "TPS22929D" H 2600 4150 60  0000 C CNN
+F 2 "" H 2000 4100 60  0000 C CNN
+F 3 "" H 2000 4100 60  0000 C CNN
+	1    2600 3800
+	1    0    0    -1
+$EndComp
+$Comp
+L +3V3 #PWR?
+U 1 1 55AC1039
+P 1525 3800
+F 0 "#PWR?" H 1525 3650 50  0001 C CNN
+F 1 "+3V3" H 1525 3940 50  0000 C CNN
+F 2 "" H 1525 3800 60  0000 C CNN
+F 3 "" H 1525 3800 60  0000 C CNN
+	1    1525 3800
+	1    0    0    -1
+$EndComp
+$Comp
+L C_Small C?
+U 1 1 55AC1091
+P 1950 3950
+F 0 "C?" H 1960 4020 50  0000 L CNN
+F 1 "1u" H 1960 3870 50  0000 L CNN
+F 2 "" H 1950 3950 60  0000 C CNN
+F 3 "" H 1950 3950 60  0000 C CNN
+	1    1950 3950
+	1    0    0    -1
+$EndComp
+Wire Wire Line
+	1950 4050 1950 4100
+Wire Wire Line
+	1950 4100 1950 4125
+Wire Wire Line
+	1950 4100 2150 4100
+Wire Wire Line
+	2150 3900 2100 3900
+Wire Wire Line
+	2100 3800 2100 3900
+Wire Wire Line
+	1825 3800 1950 3800
+Wire Wire Line
+	1950 3800 2100 3800
+Wire Wire Line
+	2100 3800 2150 3800
+Connection ~ 2100 3800
+Wire Wire Line
+	1950 3800 1950 3850
+Connection ~ 1950 3800
+$Comp
+L GND #PWR?
+U 1 1 55AC12A8
+P 1950 4125
+F 0 "#PWR?" H 1950 3875 50  0001 C CNN
+F 1 "GND" H 1950 3975 50  0000 C CNN
+F 2 "" H 1950 4125 60  0000 C CNN
+F 3 "" H 1950 4125 60  0000 C CNN
+	1    1950 4125
+	1    0    0    -1
+$EndComp
+Connection ~ 1950 4100
+$Comp
+L GND #PWR?
+U 1 1 55AC13C7
+P 3100 4125
+F 0 "#PWR?" H 3100 3875 50  0001 C CNN
+F 1 "GND" H 3100 3975 50  0000 C CNN
+F 2 "" H 3100 4125 60  0000 C CNN
+F 3 "" H 3100 4125 60  0000 C CNN
+	1    3100 4125
+	1    0    0    -1
+$EndComp
+Wire Wire Line
+	3100 4050 3100 4100
+Wire Wire Line
+	3100 4100 3100 4125
+Wire Wire Line
+	3100 4100 3050 4100
+$Comp
+L C_Small C?
+U 1 1 55AC1461
+P 3100 3950
+F 0 "C?" H 3110 4020 50  0000 L CNN
+F 1 "1u" H 3110 3870 50  0000 L CNN
+F 2 "" H 3100 3950 60  0000 C CNN
+F 3 "" H 3100 3950 60  0000 C CNN
+	1    3100 3950
+	1    0    0    -1
+$EndComp
+Wire Wire Line
+	3100 3750 3100 3800
+Wire Wire Line
+	3100 3800 3100 3850
+Wire Wire Line
+	3100 3800 3050 3800
+Connection ~ 3100 4100
+$Comp
+L +3.3V_A #PWR?
+U 1 1 55AC15A6
+P 3100 3750
+F 0 "#PWR?" H 3100 3710 30  0001 C CNN
+F 1 "+3.3V_A" H 3100 3860 30  0000 C CNN
+F 2 "" H 3100 3750 60  0000 C CNN
+F 3 "" H 3100 3750 60  0000 C CNN
+	1    3100 3750
+	1    0    0    -1
+$EndComp
+Connection ~ 3100 3800
+Text HLabel 2125 3600 0    39   Input ~ 0
+3.3V_A_EN
+Wire Wire Line
+	2125 3600 2150 3600
+$Comp
+L F_Small F?
+U 1 1 55AC3A0C
+P 1725 3800
+F 0 "F?" H 1685 3860 50  0000 L CNN
+F 1 "500mA" H 1605 3740 50  0000 L CNN
+F 2 "" H 1725 3800 60  0000 C CNN
+F 3 "" H 1725 3800 60  0000 C CNN
+	1    1725 3800
+	1    0    0    -1
+$EndComp
+Wire Wire Line
+	1625 3800 1525 3800
+$Comp
+L Battery BT?
+U 1 1 55ACA8E0
+P 6725 3575
+F 0 "BT?" H 6825 3625 50  0000 L CNN
+F 1 "1.4V to 3.6V" H 6825 3525 50  0000 L CNN
+F 2 "" V 6725 3615 60  0000 C CNN
+F 3 "" V 6725 3615 60  0000 C CNN
+	1    6725 3575
+	1    0    0    -1
+$EndComp
+$Comp
+L GND #PWR?
+U 1 1 55ACA99A
+P 6725 3775
+F 0 "#PWR?" H 6725 3525 50  0001 C CNN
+F 1 "GND" H 6725 3625 50  0000 C CNN
+F 2 "" H 6725 3775 60  0000 C CNN
+F 3 "" H 6725 3775 60  0000 C CNN
+	1    6725 3775
+	1    0    0    -1
+$EndComp
+Wire Wire Line
+	6725 3775 6725 3725
+Text HLabel 6825 3300 2    39   Input ~ 0
+Back_Bat
+Wire Wire Line
+	6725 3300 6725 3425
+Wire Wire Line
+	6825 3300 6725 3300
 $EndSCHEMATC

Commit message: Schematics: Minor cleanups
Other:
- note added: "Backup battery"
- note added: "Battery connector\n3V to 12V"
- note added: "Load switch on i2c modules power"
- note added: "Power supply: 5V output"
- moved on the sheet: BT?, C?, CONN?, D?, F?, L?, Q?, R?, U?

Commit message: Schematics: LEDs
Parts:
- D1: renamed from D?; value POWER -> YELLOW
- gave numbers to parts that had none: 20
Other:
- note added: "For KiCad DRC checks"
- moved on the sheet: C10, C11, C12, C13, C7, C8, C9, D1, L1, Q1, R13, R14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
