File: robocape.sch (KiCad schematic (older format))
At the start: 22 parts, among them U1 BEAGLEBONE, U2 CAT24C256W

Commit message: Schematics: Minor cleanups & ADC split between 3.3V & 5V
Parts:
- C2, R1, R19, R2, R20, R21, R22, R23, R24, R3, R4, R5, R6, R7, R8: footprint (none) -> _std:_0402
- U1: footprint (none) -> beaglebone:BEAGLEBONE
Connections:
- net ANALOG_0 renamed PWR_Voltage_Sense
- net VCC_ANALOG: no longer names the net of U1.C32 (VDD_ADC)
- no-connect marks 51 -> 52
Changed lines of the file:
@@
 F 0 "U1" H 1875 5000 60  0000 C CNN
 F 1 "BEAGLEBONE" H 2325 5000 60  0000 C CNN
-F 2 "" H 1825 5000 60  0000 C CNN
+F 2 "beaglebone:BEAGLEBONE" H 1825 5000 60  0001 C CNN
 F 3 "" H 1825 5000 60  0000 C CNN
 	2    1825 5000
@@
 F 0 "U1" H 2875 4900 60  0000 C CNN
 F 1 "BEAGLEBONE" H 3325 4900 60  0000 C CNN
-F 2 "" H 2825 4950 60  0000 C CNN
+F 2 "beaglebone:BEAGLEBONE" H 2825 4950 60  0001 C CNN
 F 3 "" H 2825 4950 60  0000 C CNN
 	3    2825 4950
@@
 F 0 "U1" H 4825 4900 60  0000 C CNN
 F 1 "BEAGLEBONE" H 5325 4900 60  0000 C CNN
-F 2 "" H 4775 4950 60  0000 C CNN
+F 2 "beaglebone:BEAGLEBONE" H 4775 4950 60  0001 C CNN
 F 3 "" H 4775 4950 60  0000 C CNN
 	4    4775 4950
@@
 F 0 "U1" H 5875 4900 60  0000 C CNN
 F 1 "BEAGLEBONE" H 6325 4900 60  0000 C CNN
-F 2 "" H 5825 4950 60  0000 C CNN
+F 2 "beaglebone:BEAGLEBONE" H 5825 4950 60  0001 C CNN
 F 3 "" H 5825 4950 60  0000 C CNN
 	5    5825 4950
@@
 F 0 "U1" H 5550 1975 60  0000 C CNN
 F 1 "BEAGLEBONE" H 5125 1975 60  0000 C CNN
-F 2 "" H 4900 2025 60  0000 C CNN
+F 2 "beaglebone:BEAGLEBONE" H 4900 2025 60  0001 C CNN
 F 3 "" H 4900 2025 60  0000 C CNN
 	1    4900 2025
@@
 F16 "UART_EXT_TX" I R 4825 6825 39
 F17 "UART_EXT_RX" I R 4825 6875 39
-F18 "VCC_ADC" I L 3850 5925 39
-F19 "ADC_0" I L 3850 5975 39
-F20 "ADC_1" I L 3850 6025 39
-F21 "ADC_2" I L 3850 6075 39
-F22 "ADC_3" I L 3850 6125 39
-F23 "ADC_4" I L 3850 6175 39
-F24 "ADC_5" I L 3850 6225 39
-F25 "ADC_6" I L 3850 6275 39
-F26 "I2C1_SDA" I R 4825 7225 39
-F27 "I2C1_SCL" I R 4825 7275 39
-F28 "SPI1_SCK" I R 4825 6975 39
-F29 "SPI1_MOSI" I R 4825 7025 39
-F30 "SPI1_MISO" I R 4825 7075 39
-F31 "SPI1_CS1" I R 4825 7125 39
+F18 "ADC_1" I L 3850 5975 39
+F19 "ADC_2" I L 3850 6025 39
+F20 "ADC_3" I L 3850 6075 39
+F21 "ADC_4" I L 3850 6125 39
+F22 "ADC_5" I L 3850 6175 39
+F23 "ADC_6" I L 3850 6225 39
+F24 "I2C1_SDA" I R 4825 7225 39
+F25 "I2C1_SCL" I R 4825 7275 39
+F26 "SPI1_SCK" I R 4825 6975 39
+F27 "SPI1_MOSI" I R 4825 7025 39
+F28 "SPI1_MISO" I R 4825 7075 39
+F29 "SPI1_CS1" I R 4825 7125 39
 $EndSheet
 $Sheet
-S 1800 7000 725  250
+S 1800 7000 725  350
 U 55A505D5
 F0 "Power" 60
@@
 F2 "3.3V_A_EN" I R 2525 7075 39
 F3 "Back_Bat" I R 2525 7175 39
+F4 "PWR_VOLTAGE_SENSE" I R 2525 7275 39
 $EndSheet
 $Comp
@@
 F 0 "U2" H 8600 2325 60  0000 C CNN
 F 1 "CAT24C256W" H 8850 3325 60  0000 C CNN
-F 2 "" H 8800 2875 60  0000 C CNN
+F 2 "" H 8800 2875 60  0001 C CNN
 F 3 "" H 8800 2875 60  0000 C CNN
 	1    8850 2925
@@
 F 0 "C2" H 8210 2945 50  0000 L CNN
 F 1 "100n" H 8210 2795 50  0000 L CNN
-F 2 "" H 8200 2875 60  0000 C CNN
+F 2 "_std:_0402" H 8200 2875 60  0001 C CNN
 F 3 "" H 8200 2875 60  0000 C CNN
 	1    8200 2875
@@
 F 0 "R1" H 7880 3245 50  0000 L CNN
 F 1 "10k" H 7880 3185 50  0000 L CNN
-F 2 "" H 7850 3225 60  0000 C CNN
+F 2 "_std:_0402" H 7850 3225 60  0001 C CNN
 F 3 "" H 7850 3225 60  0000 C CNN
 	1    7850 3225
@@
 F 0 "R4" H 9480 2595 50  0000 L CNN
 F 1 "4.7k" H 9480 2535 50  0000 L CNN
-F 2 "" H 9450 2575 60  0000 C CNN
+F 2 "_std:_0402" H 9450 2575 60  0001 C CNN
 F 3 "" H 9450 2575 60  0000 C CNN
 	1    9450 2575
@@
 F 0 "R5" H 9730 2595 50  0000 L CNN
 F 1 "4.7k" H 9730 2535 50  0000 L CNN
-F 2 "" H 9700 2575 60  0000 C CNN
+F 2 "_std:_0402" H 9700 2575 60  0001 C CNN
 F 3 "" H 9700 2575 60  0000 C CNN
 	1    9700 2575
@@
 F 0 "R6" H 9980 2595 50  0000 L CNN
 F 1 "4.7k" H 9980 2535 50  0000 L CNN
-F 2 "" H 9950 2575 60  0000 C CNN
+F 2 "_std:_0402" H 9950 2575 60  0001 C CNN
 F 3 "" H 9950 2575 60  0000 C CNN
 	1    9950 2575
@@
 F 0 "R7" V 10250 2700 39  0000 R CNN
 F 1 "0" V 10200 2775 39  0000 C CNN
-F 2 "" H 10200 2775 60  0000 C CNN
+F 2 "_std:_0402" H 10200 2775 60  0001 C CNN
 F 3 "" H 10200 2775 60  0000 C CNN
 	1    10200 2775
@@
 F 0 "R8" V 10250 2800 39  0000 R CNN
 F 1 "0" V 10200 2875 39  0000 C CNN
-F 2 "" H 10200 2875 60  0000 C CNN
+F 2 "_std:_0402" H 10200 2875 60  0001 C CNN
 F 3 "" H 10200 2875 60  0000 C CNN
 	1    10200 2875
@@
 F 0 "JP1" H 7850 3605 50  0000 C CNN
 F 1 "Jumper_NC_Small" H 7860 3465 50  0001 C CNN
-F 2 "" H 7850 3525 60  0000 C CNN
+F 2 "" H 7850 3525 60  0001 C CNN
 F 3 "" H 7850 3525 60  0000 C CNN
 	1    7850 3525
@@
 F 0 "R2" H 9305 1345 50  0000 L CNN
 F 1 "4.7k" H 9305 1285 50  0000 L CNN
-F 2 "" H 9275 1325 60  0000 C CNN
+F 2 "_std:_0402" H 9275 1325 60  0001 C CNN
 F 3 "" H 9275 1325 60  0000 C CNN
 	1    9275 1325
@@
 F 0 "R3" H 9555 1345 50  0000 L CNN
 F 1 "4.7k" H 9555 1285 50  0000 L CNN
-F 2 "" H 9525 1325 60  0000 C CNN
+F 2 "_std:_0402" H 9525 1325 60  0001 C CNN
 F 3 "" H 9525 1325 60  0000 C CNN
 	1    9525 1325
@@
 Text Label 4375 4300 2    39   ~ 0
 ANALOG_4
-Text Label 4375 4400 2    39   ~ 0
-ANALOG_6
 Text Label 4375 4500 2    39   ~ 0
 ANALOG_2
-Text Label 4375 4600 2    39   ~ 0
-ANALOG_0
 $Comp
 L GND #PWR016
@@
 	1    0    0    -1
 $EndComp
-Text Label 6225 4200 0    39   ~ 0
-VCC_ANALOG
+Text Label 3800 6125 2    39   ~ 0
+ANALOG_4
+Text Label 3800 6225 2    39   ~ 0
+ANALOG_6
+Text Label 3800 6025 2    39   ~ 0
+ANALOG_2
+Text Label 3800 6075 2    39   ~ 0
+ANALOG_3
 Text Label 3800 6175 2    39   ~ 0
-ANALOG_4
-Text Label 3800 6275 2    39   ~ 0
-ANALOG_6
-Text Label 3800 6075 2    39   ~ 0
-ANALOG_2
-Text Label 3800 5975 2    39   ~ 0
-ANALOG_0
-Text Label 3800 6025 2    39   ~ 0
-ANALOG_1
-Text Label 3800 6125 2    39   ~ 0
-ANALOG_3
-Text Label 3800 6225 2    39   ~ 0
 ANALOG_5
-Text Label 3800 5925 2    39   ~ 0
-VCC_ANALOG
 $Comp
 L +3.3V_A #PWR017
@@
 F 0 "D2" H 9100 5100 50  0000 C CNN
 F 1 "WHITE" H 9100 4900 50  0000 C CNN
-F 2 "" H 9100 5000 60  0000 C CNN
+F 2 "" H 9100 5000 60  0001 C CNN
 F 3 "" H 9100 5000 60  0000 C CNN
 	1    9100 5000
@@
 F 0 "D3" H 9100 5450 50  0000 C CNN
 F 1 "GREEN" H 9100 5250 50  0000 C CNN
-F 2 "" H 9100 5350 60  0000 C CNN
+F 2 "" H 9100 5350 60  0001 C CNN
 F 3 "" H 9100 5350 60  0000 C CNN
 	1    9100 5350
@@
 F 0 "D4" H 9100 5775 50  0000 C CNN
 F 1 "BLUE" H 9100 5575 50  0000 C CNN
-F 2 "" H 9100 5675 60  0000 C CNN
+F 2 "" H 9100 5675 60  0001 C CNN
 F 3 "" H 9100 5675 60  0000 C CNN
 	1    9100 5675
@@
 F 0 "D5" H 9100 6125 50  0000 C CNN
 F 1 "RED" H 9100 5925 50  0000 C CNN
-F 2 "" H 9100 6025 60  0000 C CNN
+F 2 "" H 9100 6025 60  0001 C CNN
 F 3 "" H 9100 6025 60  0000 C CNN
 	1    9100 6025
@@
 F 0 "R19" V 9630 5000 50  0000 C CNN
 F 1 "1k" V 9550 5000 50  0000 C CNN
-F 2 "" V 9480 5000 30  0000 C CNN
+F 2 "_std:_0402" V 9480 5000 30  0001 C CNN
 F 3 "" H 9550 5000 30  0000 C CNN
 	1    9550 5000
@@
 F 0 "R20" V 9630 5350 50  0000 C CNN
 F 1 "1k" V 9550 5350 50  0000 C CNN
-F 2 "" V 9480 5350 30  0000 C CNN
+F 2 "_std:_0402" V 9480 5350 30  0001 C CNN
 F 3 "" H 9550 5350 30  0000 C CNN
 	1    9550 5350
@@
 F 0 "R21" V 9630 5675 50  0000 C CNN
 F 1 "1k" V 9550 5675 50  0000 C CNN
-F 2 "" V 9480 5675 30  0000 C CNN
+F 2 "_std:_0402" V 9480 5675 30  0001 C CNN
 F 3 "" H 9550 5675 30  0000 C CNN
 	1    9550 5675
@@
 F 0 "R22" V 9630 6025 50  0000 C CNN
 F 1 "1k" V 9550 6025 50  0000 C CNN
-F 2 "" V 9480 6025 30  0000 C CNN
+F 2 "_std:_0402" V 9480 6025 30  0001 C CNN
 F 3 "" H 9550 6025 30  0000 C CNN
 	1    9550 6025
@@
 F 0 "R23" H 10380 1345 50  0000 L CNN
 F 1 "4.7k" H 10380 1285 50  0000 L CNN
-F 2 "" H 10350 1325 60  0000 C CNN
+F 2 "_std:_0402" H 10350 1325 60  0001 C CNN
 F 3 "" H 10350 1325 60  0000 C CNN
 	1    10350 1325
@@
 F 0 "R24" H 10630 1345 50  0000 L CNN
 F 1 "4.7k" H 10630 1285 50  0000 L CNN
-F 2 "" H 10600 1325 60  0000 C CNN
+F 2 "_std:_0402" H 10600 1325 60  0001 C CNN
 F 3 "" H 10600 1325 60  0000 C CNN
 	1    10600 1325
@@
 	6675 4300 6175 4300
 Wire Wire Line
-	6225 4200 6175 4200
-Wire Wire Line
-	3800 5925 3850 5925
-Wire Wire Line
-	3800 6275 3850 6275
-Wire Wire Line
 	3800 6225 3850 6225
 Wire Wire Line
@@
 	3800 6125 3850 6125
 Wire Wire Line
-	3850 6075 3800 6075
-Wire Wire Line
-	3800 6025 3850 6025
-Wire Wire Line
-	3850 5975 3800 5975
+	3800 6075 3850 6075
+Wire Wire Line
+	3850 6025 3800 6025
+Wire Wire Line
+	3800 5975 3850 5975
 Wire Notes Line
 	7375 475  7375 6550
@@
 Wire Wire Line
 	4825 7125 4875 7125
+NoConn ~ 6175 4200
+Text Label 2575 7275 0    39   ~ 0
+PWR_Voltage_Sense
+Text Label 4375 4400 2    39   ~ 0
+ANALOG_6
+Text Label 3800 5975 2    39   ~ 0
+ANALOG_1
+Wire Wire Line
+	2575 7275 2525 7275
+Text Label 4375 4600 2    39   ~ 0
+PWR_Voltage_Sense
 $EndSCHEMATC

Commit message: Netlist
Parts:
- C2: footprint _std:_0402 -> Capacitors_SMD:C_0402
- D2, D3, D4, D5: footprint (none) -> LEDs:LED-0603
- JP1: footprint (none) -> Pin_Headers:Pin_Header_Straight_1x02
- R1, R19, R2, R20, R21, R22, R23, R24, R3, R4, R5, R6, R7, R8: footprint _std:_0402 -> Resistors_SMD:R_0402
- U2: footprint (none) -> SMD_Packages:SOIC-8-N
