File: robocape.sch (KiCad schematic (older format))
At the start: 22 parts, among them U1 BEAGLEBONE, U2 CAT24C256W

Commit message: Schematics: CAN termination resistor + PWM gen decoupling cap
Parts:
- U1: footprint beaglebone:BEAGLEBONE -> _beaglebone:BEAGLEBONE
Changed lines of the file:
@@
 F 0 "U1" H 1875 5000 60  0000 C CNN
 F 1 "BEAGLEBONE" H 2325 5000 60  0000 C CNN
-F 2 "beaglebone:BEAGLEBONE" H 1825 5000 60  0001 C CNN
+F 2 "_beaglebone:BEAGLEBONE" H 1825 5000 60  0001 C CNN
 F 3 "" H 1825 5000 60  0000 C CNN
 	2    1825 5000
@@
 F 0 "U1" H 2875 4900 60  0000 C CNN
 F 1 "BEAGLEBONE" H 3325 4900 60  0000 C CNN
-F 2 "beaglebone:BEAGLEBONE" H 2825 4950 60  0001 C CNN
+F 2 "_beaglebone:BEAGLEBONE" H 2825 4950 60  0001 C CNN
 F 3 "" H 2825 4950 60  0000 C CNN
 	3    2825 4950
@@
 F 0 "U1" H 4825 4900 60  0000 C CNN
 F 1 "BEAGLEBONE" H 5325 4900 60  0000 C CNN
-F 2 "beaglebone:BEAGLEBONE" H 4775 4950 60  0001 C CNN
+F 2 "_beaglebone:BEAGLEBONE" H 4775 4950 60  0001 C CNN
 F 3 "" H 4775 4950 60  0000 C CNN
 	4    4775 4950
@@
 F 0 "U1" H 5875 4900 60  0000 C CNN
 F 1 "BEAGLEBONE" H 6325 4900 60  0000 C CNN
-F 2 "beaglebone:BEAGLEBONE" H 5825 4950 60  0001 C CNN
+F 2 "_beaglebone:BEAGLEBONE" H 5825 4950 60  0001 C CNN
 F 3 "" H 5825 4950 60  0000 C CNN
 	5    5825 4950
@@
 F 0 "U1" H 5550 1975 60  0000 C CNN
 F 1 "BEAGLEBONE" H 5125 1975 60  0000 C CNN
-F 2 "beaglebone:BEAGLEBONE" H 4900 2025 60  0001 C CNN
+F 2 "_beaglebone:BEAGLEBONE" H 4900 2025 60  0001 C CNN
 F 3 "" H 4900 2025 60  0000 C CNN
 	1    4900 2025
