File: sensors.sch (KiCad schematic (older format))
At the start: 18 parts, among them J1 SMA, U10 MPU-9250, U11 MS5611-01BA, U3 BQ32000, U9 MAX-M8, X1 32768Hz

Commit message: Schematics: Minor cleanups & ADC split between 3.3V & 5V
Parts:
- C1, C16, C17, C18, C19, C20, C21, C3, C4, C5, R17, R18: footprint (none) -> _std:_0402
- U11: footprint MODULE -> _sensors:_MS5611-01BA
Changed lines of the file:
@@
 F 0 "U10" H 3700 3050 60  0000 C CNN
 F 1 "MPU-9250" H 3050 3050 60  0000 C CNN
-F 2 "" H 3300 2850 60  0000 C CNN
+F 2 "" H 3300 2850 60  0001 C CNN
 F 3 "" H 3300 2850 60  0000 C CNN
 	1    3300 2250
@@
 NoConn ~ 2500 2150
 $Comp
-L +3.3V_A #PWR078
+L +3.3V_A #PWR082
 U 1 1 55A53AEE
 P 2000 1575
-F 0 "#PWR078" H 2000 1535 30  0001 C CNN
+F 0 "#PWR082" H 2000 1535 30  0001 C CNN
 F 1 "+3.3V_A" H 2000 1685 30  0000 C CNN
 F 2 "" H 2000 1575 60  0000 C CNN
@@
 Connection ~ 2450 1600
 $Comp
-L GND #PWR079
+L GND #PWR083
 U 1 1 55A53B15
 P 2000 1925
-F 0 "#PWR079" H 2000 1675 50  0001 C CNN
+F 0 "#PWR083" H 2000 1675 50  0001 C CNN
 F 1 "GND" H 2000 1775 50  0000 C CNN
 F 2 "" H 2000 1925 60  0000 C CNN
@@
 F 0 "C18" H 2285 1820 50  0000 L CNN
 F 1 "10n" H 2285 1670 50  0000 L CNN
-F 2 "" H 2275 1750 60  0000 C CNN
+F 2 "_std:_0402" H 2275 1750 60  0001 C CNN
 F 3 "" H 2275 1750 60  0000 C CNN
 	1    2275 1750
@@
 F 0 "C17" H 2010 1820 50  0000 L CNN
 F 1 "100n" H 2010 1670 50  0000 L CNN
-F 2 "" H 2000 1750 60  0000 C CNN
+F 2 "_std:_0402" H 2000 1750 60  0001 C CNN
 F 3 "" H 2000 1750 60  0000 C CNN
 	1    2000 1750
@@
 F 0 "C20" H 4585 2670 50  0000 L CNN
 F 1 "100n" H 4585 2520 50  0000 L CNN
-F 2 "" H 4575 2600 60  0000 C CNN
+F 2 "_std:_0402" H 4575 2600 60  0001 C CNN
 F 3 "" H 4575 2600 60  0000 C CNN
 	1    4575 2600
@@
 NoConn ~ 4100 2750
 $Comp
-L +3.3V_A #PWR080
+L +3.3V_A #PWR084
 U 1 1 55A53F56
 P 4275 2850
-F 0 "#PWR080" H 4275 2810 30  0001 C CNN
+F 0 "#PWR084" H 4275 2810 30  0001 C CNN
 F 1 "+3.3V_A" H 4275 2960 30  0000 C CNN
 F 2 "" H 4275 2850 60  0000 C CNN
@@
 	4275 2850 4100 2850
 $Comp
-L GND #PWR081
+L GND #PWR085
 U 1 1 55A53F96
 P 4275 2950
-F 0 "#PWR081" H 4275 2700 50  0001 C CNN
+F 0 "#PWR085" H 4275 2700 50  0001 C CNN
 F 1 "GND" H 4275 2800 50  0000 C CNN
 F 2 "" H 4275 2950 60  0000 C CNN
@@
 	4275 2950 4100 2950
 $Comp
-L GND #PWR082
+L GND #PWR086
 U 1 1 55A53FE1
 P 4575 2750
-F 0 "#PWR082" H 4575 2500 50  0001 C CNN
+F 0 "#PWR086" H 4575 2500 50  0001 C CNN
 F 1 "GND" H 4575 2600 50  0000 C CNN
 F 2 "" H 4575 2750 60  0000 C CNN
@@
 F 0 "U11" H 8675 2575 50  0000 C CNN
 F 1 "MS5611-01BA" H 8175 2575 50  0000 C CNN
-F 2 "MODULE" H 8325 2175 50  0001 C CNN
+F 2 "_sensors:_MS5611-01BA" H 8325 2175 50  0001 C CNN
 F 3 "DOCUMENTATION" H 8325 2175 50  0001 C CNN
 	1    8325 2175
@@
 NoConn ~ 9075 2175
 $Comp
-L GND #PWR083
+L GND #PWR087
 U 1 1 55A56310
 P 9125 2425
-F 0 "#PWR083" H 9125 2175 50  0001 C CNN
+F 0 "#PWR087" H 9125 2175 50  0001 C CNN
 F 1 "GND" H 9125 2275 50  0000 C CNN
 F 2 "" H 9125 2425 60  0000 C CNN
@@
 	9075 2075 9125 2075
 $Comp
-L +3.3V_A #PWR084
+L +3.3V_A #PWR088
 U 1 1 55A56473
 P 7400 1925
-F 0 "#PWR084" H 7400 1885 30  0001 C CNN
+F 0 "#PWR088" H 7400 1885 30  0001 C CNN
 F 1 "+3.3V_A" H 7400 2035 30  0000 C CNN
 F 2 "" H 7400 1925 60  0000 C CNN
@@
 F 0 "C21" H 7410 2295 50  0000 L CNN
 F 1 "100n" H 7410 2145 50  0000 L CNN
-F 2 "" H 7400 2225 60  0000 C CNN
+F 2 "_std:_0402" H 7400 2225 60  0001 C CNN
 F 3 "" H 7400 2225 60  0000 C CNN
 	1    7400 2225
@@
 Connection ~ 7400 1975
 $Comp
-L GND #PWR085
+L GND #PWR089
 U 1 1 55A566F0
 P 7400 2425
-F 0 "#PWR085" H 7400 2175 50  0001 C CNN
+F 0 "#PWR089" H 7400 2175 50  0001 C CNN
 F 1 "GND" H 7400 2275 50  0000 C CNN
 F 2 "" H 7400 2425 60  0000 C CNN
@@
 I2C address: 0x77\n
 $Comp
-L +3V3 #PWR086
+L +3V3 #PWR090
 U 1 1 55AC52F9
 P 1825 5000
-F 0 "#PWR086" H 1825 4850 50  0001 C CNN
+F 0 "#PWR090" H 1825 4850 50  0001 C CNN
 F 1 "+3V3" H 1825 5140 50  0000 C CNN
 F 2 "" H 1825 5000 60  0000 C CNN
@@
 	2325 5350 2575 5350
 $Comp
-L GND #PWR087
+L GND #PWR091
 U 1 1 55AC5654
 P 2525 6500
-F 0 "#PWR087" H 2525 6250 50  0001 C CNN
+F 0 "#PWR091" H 2525 6250 50  0001 C CNN
 F 1 "GND" H 2525 6350 50  0000 C CNN
 F 2 "" H 2525 6500 60  0000 C CNN
@@
 F 0 "U9" H 3575 4200 60  0000 C CNN
 F 1 "MAX-M8" H 3225 5900 60  0000 C CNN
-F 2 "" H 4075 5850 60  0000 C CNN
+F 2 "" H 4075 5850 60  0001 C CNN
 F 3 "" H 4075 5850 60  0000 C CNN
 	1    3225 5400
@@
 F 0 "R17" V 4025 5525 50  0000 L CNN
 F 1 "330" V 4075 5450 39  0000 C CNN
-F 2 "" H 4075 5450 60  0000 C CNN
+F 2 "_std:_0402" H 4075 5450 60  0001 C CNN
 F 3 "" H 4075 5450 60  0000 C CNN
 	1    4075 5450
@@
 F 0 "R18" V 4025 5625 50  0000 L CNN
 F 1 "330" V 4075 5550 39  0000 C CNN
-F 2 "" H 4075 5550 60  0000 C CNN
+F 2 "_std:_0402" H 4075 5550 60  0001 C CNN
 F 3 "" H 4075 5550 60  0000 C CNN
 	1    4075 5550
@@
 F 0 "C16" H 1835 5270 50  0000 L CNN
 F 1 "0.1u" H 1835 5120 50  0000 L CNN
-F 2 "" H 1825 5200 60  0000 C CNN
+F 2 "_std:_0402" H 1825 5200 60  0001 C CNN
 F 3 "" H 1825 5200 60  0000 C CNN
 	1    1825 5200
@@
 Connection ~ 1825 5050
 $Comp
-L GND #PWR088
+L GND #PWR092
 U 1 1 55AC69AE
 P 1825 5650
-F 0 "#PWR088" H 1825 5400 50  0001 C CNN
+F 0 "#PWR092" H 1825 5400 50  0001 C CNN
 F 1 "GND" H 1825 5500 50  0000 C CNN
 F 2 "" H 1825 5650 60  0000 C CNN
@@
 F 0 "C19" H 2385 5570 50  0000 L CNN
 F 1 "0.1u" H 2385 5420 50  0000 L CNN
-F 2 "" H 2375 5500 60  0000 C CNN
+F 2 "_std:_0402" H 2375 5500 60  0001 C CNN
 F 3 "" H 2375 5500 60  0000 C CNN
 	1    2375 5500
@@
 $EndComp
 $Comp
-L GND #PWR089
+L GND #PWR093
 U 1 1 55B15C94
 P 4475 5000
-F 0 "#PWR089" H 4475 4750 50  0001 C CNN
+F 0 "#PWR093" H 4475 4750 50  0001 C CNN
 F 1 "GND" H 4475 4850 50  0000 C CNN
 F 2 "" H 4475 5000 60  0000 C CNN
@@
 F 0 "U3" H 8700 4300 59  0000 C CNN
 F 1 "BQ32000" H 8400 5300 59  0000 C CNN
-F 2 "" H 8400 5500 39  0000 C CNN
+F 2 "" H 8400 5500 39  0001 C CNN
 F 3 "" H 8400 5500 39  0000 C CNN
 	1    8400 4850
@@
 $EndComp
 $Comp
-L +3.3V_A #PWR090
+L +3.3V_A #PWR094
 U 1 1 55B17AA3
 P 7200 4500
-F 0 "#PWR090" H 7200 4460 30  0001 C CNN
+F 0 "#PWR094" H 7200 4460 30  0001 C CNN
 F 1 "+3.3V_A" H 7200 4610 30  0000 C CNN
 F 2 "" H 7200 4500 60  0000 C CNN
@@
 F 0 "C3" H 7760 5070 50  0000 L CNN
 F 1 "220n" H 7760 4920 50  0000 L CNN
-F 2 "" H 7750 5000 60  0000 C CNN
+F 2 "_std:_0402" H 7750 5000 60  0001 C CNN
 F 3 "" H 7750 5000 60  0000 C CNN
 	1    7750 5000
@@
 Connection ~ 7750 4850
 $Comp
-L GND #PWR091
+L GND #PWR095
 U 1 1 55B17AB9
 P 7200 5300
-F 0 "#PWR091" H 7200 5050 50  0001 C CNN
+F 0 "#PWR095" H 7200 5050 50  0001 C CNN
 F 1 "GND" H 7200 5150 50  0000 C CNN
 F 2 "" H 7200 5300 60  0000 C CNN
@@
 F 0 "C1" H 7210 5070 50  0000 L CNN
 F 1 "1u" H 7210 4920 50  0000 L CNN
-F 2 "" H 7200 5000 60  0000 C CNN
+F 2 "_std:_0402" H 7200 5000 60  0001 C CNN
 F 3 "" H 7200 5000 60  0000 C CNN
 	1    7200 5000
@@
 F 0 "X1" H 9350 5550 60  0000 C CNN
 F 1 "32768Hz" H 9350 5625 60  0000 C CNN
-F 2 "" H 9350 5450 60  0000 C CNN
+F 2 "" H 9350 5450 60  0001 C CNN
 F 3 "" H 9350 5450 60  0000 C CNN
 	1    9350 5450
@@
 	9000 5250 8950 5250
 $Comp
-L GND #PWR092
+L GND #PWR096
 U 1 1 55B17ADB
 P 9350 5800
-F 0 "#PWR092" H 9350 5550 50  0001 C CNN
+F 0 "#PWR096" H 9350 5550 50  0001 C CNN
 F 1 "GND" H 9350 5650 50  0000 C CNN
 F 2 "" H 9350 5800 60  0000 C CNN
@@
 F 0 "C5" H 9710 5670 50  0000 L CNN
 F 1 "10p" H 9710 5520 50  0000 L CNN
-F 2 "" H 9700 5600 60  0000 C CNN
+F 2 "_std:_0402" H 9700 5600 60  0001 C CNN
 F 3 "" H 9700 5600 60  0000 C CNN
 	1    9700 5600
@@
 F 0 "C4" H 9010 5670 50  0000 L CNN
 F 1 "10p" H 9010 5520 50  0000 L CNN
-F 2 "" H 9000 5600 60  0000 C CNN
+F 2 "_std:_0402" H 9000 5600 60  0001 C CNN
 F 3 "" H 9000 5600 60  0000 C CNN
 	1    9000 5600

Commit message: Netlist
Parts:
- C1, C16, C17, C18, C19, C20, C21, C3, C4, C5: footprint _std:_0402 -> Capacitors_SMD:C_0402
- J1: footprint SMA_antenna -> _connectors:SMA-CONN
- R17, R18: footprint _std:_0402 -> Resistors_SMD:R_0402
- U10: footprint (none) -> Housings_DFN_QFN:QFN-24-1EP_3x3mm_Pitch0.4mm
- U3: footprint (none) -> SMD_Packages:SOIC-8-N
- U9: footprint (none) -> _sensors:MAX-M8
- X1: footprint (none) -> _div:_TSX-3225-SMD-XTAL
Changed lines of the file:
@@
 F 0 "U10" H 3700 3050 60  0000 C CNN
 F 1 "MPU-9250" H 3050 3050 60  0000 C CNN
-F 2 "" H 3300 2850 60  0001 C CNN
+F 2 "Housings_DFN_QFN:QFN-24-1EP_3x3mm_Pitch0.4mm" H 3300 2850 60  0001 C CNN
 F 3 "" H 3300 2850 60  0000 C CNN
 	1    3300 2250
@@
 NoConn ~ 2500 2150
 $Comp
-L +3.3V_A #PWR80
+L +3.3V_A #PWR083
 U 1 1 55A53AEE
 P 2000 1575
-F 0 "#PWR80" H 2000 1535 30  0001 C CNN
+F 0 "#PWR083" H 2000 1535 30  0001 C CNN
 F 1 "+3.3V_A" H 2000 1685 30  0000 C CNN
 F 2 "" H 2000 1575 60  0000 C CNN
@@
 Connection ~ 2450 1600
 $Comp
-L GND #PWR81
+L GND #PWR084
 U 1 1 55A53B15
 P 2000 1925
-F 0 "#PWR81" H 2000 1675 50  0001 C CNN
+F 0 "#PWR084" H 2000 1675 50  0001 C CNN
 F 1 "GND" H 2000 1775 50  0000 C CNN
 F 2 "" H 2000 1925 60  0000 C CNN
@@
 F 0 "C18" H 2285 1820 50  0000 L CNN
 F 1 "10n" H 2285 1670 50  0000 L CNN
-F 2 "_std:_0402" H 2275 1750 60  0001 C CNN
+F 2 "Capacitors_SMD:C_0402" H 2275 1750 60  0001 C CNN
 F 3 "" H 2275 1750 60  0000 C CNN
 	1    2275 1750
@@
 F 0 "C17" H 2010 1820 50  0000 L CNN
 F 1 "100n" H 2010 1670 50  0000 L CNN
-F 2 "_std:_0402" H 2000 1750 60  0001 C CNN
+F 2 "Capacitors_SMD:C_0402" H 2000 1750 60  0001 C CNN
 F 3 "" H 2000 1750 60  0000 C CNN
 	1    2000 1750
@@
 F 0 "C20" H 4585 2670 50  0000 L CNN
 F 1 "100n" H 4585 2520 50  0000 L CNN
-F 2 "_std:_0402" H 4575 2600 60  0001 C CNN
+F 2 "Capacitors_SMD:C_0402" H 4575 2600 60  0001 C CNN
 F 3 "" H 4575 2600 60  0000 C CNN
 	1    4575 2600
@@
 NoConn ~ 4100 2750
 $Comp
-L +3.3V_A #PWR83
+L +3.3V_A #PWR085
 U 1 1 55A53F56
 P 4275 2850
-F 0 "#PWR83" H 4275 2810 30  0001 C CNN
+F 0 "#PWR085" H 4275 2810 30  0001 C CNN
 F 1 "+3.3V_A" H 4275 2960 30  0000 C CNN
 F 2 "" H 4275 2850 60  0000 C CNN
@@
 	4275 2850 4100 2850
 $Comp
-L GND #PWR84
+L GND #PWR086
 U 1 1 55A53F96
 P 4275 2950
-F 0 "#PWR84" H 4275 2700 50  0001 C CNN
+F 0 "#PWR086" H 4275 2700 50  0001 C CNN
 F 1 "GND" H 4275 2800 50  0000 C CNN
 F 2 "" H 4275 2950 60  0000 C CNN
@@
 	4275 2950 4100 2950
 $Comp
-L GND #PWR86
+L GND #PWR087
 U 1 1 55A53FE1
 P 4575 2750
-F 0 "#PWR86" H 4575 2500 50  0001 C CNN
+F 0 "#PWR087" H 4575 2500 50  0001 C CNN
 F 1 "GND" H 4575 2600 50  0000 C CNN
 F 2 "" H 4575 2750 60  0000 C CNN
@@
 NoConn ~ 9075 2175
 $Comp
-L GND #PWR91
+L GND #PWR088
 U 1 1 55A56310
 P 9125 2425
-F 0 "#PWR91" H 9125 2175 50  0001 C CNN
+F 0 "#PWR088" H 9125 2175 50  0001 C CNN
 F 1 "GND" H 9125 2275 50  0000 C CNN
 F 2 "" H 9125 2425 60  0000 C CNN
@@
 	9075 2075 9125 2075
 $Comp
-L +3.3V_A #PWR89
+L +3.3V_A #PWR089
 U 1 1 55A56473
 P 7400 1925
-F 0 "#PWR89" H 7400 1885 30  0001 C CNN
+F 0 "#PWR089" H 7400 1885 30  0001 C CNN
 F 1 "+3.3V_A" H 7400 2035 30  0000 C CNN
 F 2 "" H 7400 1925 60  0000 C CNN
@@
 F 0 "C21" H 7410 2295 50  0000 L CNN
 F 1 "100n" H 7410 2145 50  0000 L CNN
-F 2 "_std:_0402" H 7400 2225 60  0001 C CNN
+F 2 "Capacitors_SMD:C_0402" H 7400 2225 60  0001 C CNN
 F 3 "" H 7400 2225 60  0000 C CNN
 	1    7400 2225
@@
 Connection ~ 7400 1975
 $Comp
-L GND #PWR90
+L GND #PWR090
 U 1 1 55A566F0
 P 7400 2425
-F 0 "#PWR90" H 7400 2175 50  0001 C CNN
+F 0 "#PWR090" H 7400 2175 50  0001 C CNN
 F 1 "GND" H 7400 2275 50  0000 C CNN
 F 2 "" H 7400 2425 60  0000 C CNN
@@
 I2C address: 0x77\n
 $Comp
-L +3V3 #PWR78
+L +3V3 #PWR091
 U 1 1 55AC52F9
 P 1825 5000
-F 0 "#PWR78" H 1825 4850 50  0001 C CNN
+F 0 "#PWR091" H 1825 4850 50  0001 C CNN
 F 1 "+3V3" H 1825 5140 50  0000 C CNN
 F 2 "" H 1825 5000 60  0000 C CNN
@@
 	2325 5350 2575 5350
 $Comp
-L GND #PWR82
+L GND #PWR092
 U 1 1 55AC5654
 P 2525 6500
-F 0 "#PWR82" H 2525 6250 50  0001 C CNN
+F 0 "#PWR092" H 2525 6250 50  0001 C CNN
 F 1 "GND" H 2525 6350 50  0000 C CNN
 F 2 "" H 2525 6500 60  0000 C CNN
@@
 F 0 "U9" H 3575 4200 60  0000 C CNN
 F 1 "MAX-M8" H 3225 5900 60  0000 C CNN
-F 2 "" H 4075 5850 60  0001 C CNN
+F 2 "_sensors:MAX-M8" H 4075 5850 60  0001 C CNN
 F 3 "" H 4075 5850 60  0000 C CNN
 	1    3225 5400
@@
 F 0 "R17" V 4025 5525 50  0000 L CNN
 F 1 "330" V 4075 5450 39  0000 C CNN
-F 2 "_std:_0402" H 4075 5450 60  0001 C CNN
+F 2 "Resistors_SMD:R_0402" H 4075 5450 60  0001 C CNN
 F 3 "" H 4075 5450 60  0000 C CNN
 	1    4075 5450
@@
 F 0 "R18" V 4025 5625 50  0000 L CNN
 F 1 "330" V 4075 5550 39  0000 C CNN
-F 2 "_std:_0402" H 4075 5550 60  0001 C CNN
+F 2 "Resistors_SMD:R_0402" H 4075 5550 60  0001 C CNN
 F 3 "" H 4075 5550 60  0000 C CNN
 	1    4075 5550
@@
 F 0 "C16" H 1835 5270 50  0000 L CNN
 F 1 "0.1u" H 1835 5120 50  0000 L CNN
-F 2 "_std:_0402" H 1825 5200 60  0001 C CNN
+F 2 "Capacitors_SMD:C_0402" H 1825 5200 60  0001 C CNN
 F 3 "" H 1825 5200 60  0000 C CNN
 	1    1825 5200
@@
 Connection ~ 1825 5050
 $Comp
-L GND #PWR79
+L GND #PWR093
 U 1 1 55AC69AE
 P 1825 5650
-F 0 "#PWR79" H 1825 5400 50  0001 C CNN
+F 0 "#PWR093" H 1825 5400 50  0001 C CNN
 F 1 "GND" H 1825 5500 50  0000 C CNN
 F 2 "" H 1825 5650 60  0000 C CNN
@@
 F 0 "C19" H 2385 5570 50  0000 L CNN
 F 1 "0.1u" H 2385 5420 50  0000 L CNN
-F 2 "_std:_0402" H 2375 5500 60  0001 C CNN
+F 2 "Capacitors_SMD:C_0402" H 2375 5500 60  0001 C CNN
 F 3 "" H 2375 5500 60  0000 C CNN
 	1    2375 5500
@@
 F 0 "J1" H 4625 5365 60  0000 C CNN
 F 1 "SMA" H 4690 5290 60  0000 C CNN
-F 2 "SMA_antenna" H 4500 5500 50  0000 C CNN
+F 2 "_connectors:SMA-CONN" H 4500 5500 50  0000 C CNN
 F 3 "" H 4500 5050 60  0000 C CNN
 	1    4500 5050
@@
 $EndComp
 $Comp
-L GND #PWR85
+L GND #PWR094
 U 1 1 55B15C94
 P 4475 5000
-F 0 "#PWR85" H 4475 4750 50  0001 C CNN
+F 0 "#PWR094" H 4475 4750 50  0001 C CNN
 F 1 "GND" H 4475 4850 50  0000 C CNN
 F 2 "" H 4475 5000 60  0000 C CNN
@@
 F 0 "U3" H 8700 4300 59  0000 C CNN
 F 1 "BQ32000" H 8400 5300 59  0000 C CNN
-F 2 "" H 8400 5500 39  0001 C CNN
+F 2 "SMD_Packages:SOIC-8-N" H 8400 5500 39  0001 C CNN
 F 3 "" H 8400 5500 39  0000 C CNN
 	1    8400 4850
@@
 $EndComp
 $Comp
-L +3.3V_A #PWR87
+L +3.3V_A #PWR095
 U 1 1 55B17AA3
 P 7200 4500
-F 0 "#PWR87" H 7200 4460 30  0001 C CNN
+F 0 "#PWR095" H 7200 4460 30  0001 C CNN
 F 1 "+3.3V_A" H 7200 4610 30  0000 C CNN
 F 2 "" H 7200 4500 60  0000 C CNN
@@
 F 0 "C3" H 7760 5070 50  0000 L CNN
 F 1 "220n" H 7760 4920 50  0000 L CNN
-F 2 "_std:_0402" H 7750 5000 60  0001 C CNN
+F 2 "Capacitors_SMD:C_0402" H 7750 5000 60  0001 C CNN
 F 3 "" H 7750 5000 60  0000 C CNN
 	1    7750 5000
@@
 Connection ~ 7750 4850
 $Comp
-L GND #PWR88
+L GND #PWR096
 U 1 1 55B17AB9
 P 7200 5300
-F 0 "#PWR88" H 7200 5050 50  0001 C CNN
+F 0 "#PWR096" H 7200 5050 50  0001 C CNN
 F 1 "GND" H 7200 5150 50  0000 C CNN
 F 2 "" H 7200 5300 60  0000 C CNN
@@
 F 0 "C1" H 7210 5070 50  0000 L CNN
 F 1 "1u" H 7210 4920 50  0000 L CNN
-F 2 "_std:_0402" H 7200 5000 60  0001 C CNN
+F 2 "Capacitors_SMD:C_0402" H 7200 5000 60  0001 C CNN
 F 3 "" H 7200 5000 60  0000 C CNN
 	1    7200 5000
@@
 F 0 "X1" H 9350 5550 60  0000 C CNN
 F 1 "32768Hz" H 9350 5625 60  0000 C CNN
-F 2 "" H 9350 5450 60  0001 C CNN
+F 2 "_div:_TSX-3225-SMD-XTAL" H 9350 5450 60  0001 C CNN
 F 3 "" H 9350 5450 60  0000 C CNN
 	1    9350 5450
@@
 	9000 5250 8950 5250
 $Comp
-L GND #PWR92
+L GND #PWR097
 U 1 1 55B17ADB
 P 9350 5800
-F 0 "#PWR92" H 9350 5550 50  0001 C CNN
+F 0 "#PWR097" H 9350 5550 50  0001 C CNN
 F 1 "GND" H 9350 5650 50  0000 C CNN
 F 2 "" H 9350 5800 60  0000 C CNN
@@
 F 0 "C5" H 9710 5670 50  0000 L CNN
 F 1 "10p" H 9710 5520 50  0000 L CNN
-F 2 "_std:_0402" H 9700 5600 60  0001 C CNN
+F 2 "Capacitors_SMD:C_0402" H 9700 5600 60  0001 C CNN
 F 3 "" H 9700 5600 60  0000 C CNN
 	1    9700 5600
@@
 F 0 "C4" H 9010 5670 50  0000 L CNN
 F 1 "10p" H 9010 5520 50  0000 L CNN
-F 2 "_std:_0402" H 9000 5600 60  0001 C CNN
+F 2 "Capacitors_SMD:C_0402" H 9000 5600 60  0001 C CNN
 F 3 "" H 9000 5600 60  0000 C CNN
 	1    9000 5600

Commit message: PCB: More and more tracks
Parts:
- removed U10: MPU-9250, Housings_DFN_QFN:QFN-24-1EP_3x3mm_Pitch0.4mm, symbol MPU-9250
- added U?: MPU-9250, symbol MPU-9250
Connections:
- net +3.3V_A: now also U?.13 (VDD), U?.19 (RESV), U?.8 (VDDIO)
- net GND: now also U?.18 (GND), U?.20 (RESV), U?.25 (GND)
- net MPU9250_CS: now also U?.22 (nCS)
- net MPU9250_INT: now also U?.12 (INT)
- net MPU9250_MISO: now also U?.9 (AD0/SD0)
- net MPU9250_MOSI: now also U?.24 (SDA/SDI)
- net MPU9250_SCK: now also U?.23 (SCL/SCLK)
- net at C20.1: now also U?.10 (REGOUT)
Changed lines of the file:
@@
 Comment4 ""
 $EndDescr
-$Comp
-L MPU-9250 U10
-U 1 1 55A53A6C
-P 3300 2250
-F 0 "U10" H 3700 3050 60  0000 C CNN
-F 1 "MPU-9250" H 3050 3050 60  0000 C CNN
-F 2 "Housings_DFN_QFN:QFN-24-1EP_3x3mm_Pitch0.4mm" H 3300 2850 60  0001 C CNN
-F 3 "" H 3300 2850 60  0000 C CNN
-	1    3300 2250
-	1    0    0    -1
-$EndComp
 NoConn ~ 2500 2950
 NoConn ~ 2500 2850
@@
 Wire Wire Line
 	7675 4750 7750 4750
+$Comp
+L MPU-9250 U?
+U 1 1 55B15A2B
+P 3300 2250
+F 0 "U?" H 3700 3050 60  0000 C CNN
+F 1 "MPU-9250" H 3050 3050 60  0000 C CNN
+F 2 "" H 3300 2850 60  0000 C CNN
+F 3 "" H 3300 2850 60  0000 C CNN
+	1    3300 2250
+	1    0    0    -1
+$EndComp
 $EndSCHEMATC

Commit message: PCB: Done
Parts:
- U10: renamed from U?; footprint (none) -> Housings_DFN_QFN:QFN-24-1EP_3x3mm_Pitch0.4mm
Changed lines of the file:
@@
 	7675 4750 7750 4750
 $Comp
-L MPU-9250 U?
+L MPU-9250 U10
 U 1 1 55B15A2B
 P 3300 2250
-F 0 "U?" H 3700 3050 60  0000 C CNN
+F 0 "U10" H 3700 3050 60  0000 C CNN
 F 1 "MPU-9250" H 3050 3050 60  0000 C CNN
-F 2 "" H 3300 2850 60  0000 C CNN
+F 2 "Housings_DFN_QFN:QFN-24-1EP_3x3mm_Pitch0.4mm" H 3300 2850 60  0001 C CNN
 F 3 "" H 3300 2850 60  0000 C CNN
 	1    3300 2250
