File: connectivity.sch (KiCad schematic (older format))
At the start: 44 parts, among them SW1 SW_PUSH, U4 XBee_Header, U5 PCA9685, U6 SN65HVD232D

Commit message: PCB: Correct footprint and layout of 5V regulator
Also added some 3D models (GPS, SMA)
Parts:
- CONN18: footprint (none) -> _connectors:_Molex-PicoBlade-SMD-6
- CONN19, CONN20: footprint (none) -> _connectors:_Molex-PicoBlade-SMD-4
Changed lines of the file:
@@
 XBEE_RTS
 $Comp
-L +3V3 #PWR33
+L +3V3 #PWR029
 U 1 1 55A68A9D
 P 1625 1575
-F 0 "#PWR33" H 1625 1425 50  0001 C CNN
+F 0 "#PWR029" H 1625 1425 50  0001 C CNN
 F 1 "+3V3" H 1625 1715 50  0000 C CNN
 F 2 "" H 1625 1575 60  0000 C CNN
@@
 NoConn ~ 1675 2525
 $Comp
-L GND #PWR34
+L GND #PWR030
 U 1 1 55A68AF1
 P 1625 2875
-F 0 "#PWR34" H 1625 2625 50  0001 C CNN
+F 0 "#PWR030" H 1625 2625 50  0001 C CNN
 F 1 "GND" H 1625 2725 50  0000 C CNN
 F 2 "" H 1625 2875 60  0000 C CNN
@@
 $EndComp
 $Comp
-L GND #PWR32
+L GND #PWR031
 U 1 1 55A68BA5
 P 1150 2625
-F 0 "#PWR32" H 1150 2375 50  0001 C CNN
+F 0 "#PWR031" H 1150 2375 50  0001 C CNN
 F 1 "GND" H 1150 2475 50  0000 C CNN
 F 2 "" H 1150 2625 60  0000 C CNN
@@
 $EndComp
 $Comp
-L +3V3 #PWR31
+L +3V3 #PWR032
 U 1 1 55A68C91
 P 1150 1575
-F 0 "#PWR31" H 1150 1425 50  0001 C CNN
+F 0 "#PWR032" H 1150 1425 50  0001 C CNN
 F 1 "+3V3" H 1150 1715 50  0000 C CNN
 F 2 "" H 1150 1575 60  0000 C CNN
@@
 $EndComp
 $Comp
-L GND #PWR36
+L GND #PWR033
 U 1 1 55A7FFC8
 P 1950 6375
-F 0 "#PWR36" H 1950 6125 50  0001 C CNN
+F 0 "#PWR033" H 1950 6125 50  0001 C CNN
 F 1 "GND" H 1950 6225 50  0000 C CNN
 F 2 "" H 1950 6375 60  0000 C CNN
@@
 $EndComp
 $Comp
-L +3.3V_A #PWR35
+L +3.3V_A #PWR034
 U 1 1 55A8001C
 P 1750 4675
-F 0 "#PWR35" H 1750 4635 30  0001 C CNN
+F 0 "#PWR034" H 1750 4635 30  0001 C CNN
 F 1 "+3.3V_A" H 1750 4785 30  0000 C CNN
 F 2 "" H 1750 4675 60  0000 C CNN
@@
 POWER
 $Comp
-L GND #PWR44
+L GND #PWR035
 U 1 1 55A83C7A
 P 6650 4675
-F 0 "#PWR44" H 6650 4425 50  0001 C CNN
+F 0 "#PWR035" H 6650 4425 50  0001 C CNN
 F 1 "GND" H 6650 4525 50  0000 C CNN
 F 2 "" H 6650 4675 60  0000 C CNN
@@
 POWER
 $Comp
-L GND #PWR45
+L GND #PWR036
 U 1 1 55A83D46
 P 6650 5350
-F 0 "#PWR45" H 6650 5100 50  0001 C CNN
+F 0 "#PWR036" H 6650 5100 50  0001 C CNN
 F 1 "GND" H 6650 5200 50  0000 C CNN
 F 2 "" H 6650 5350 60  0000 C CNN
@@
 POWER
 $Comp
-L GND #PWR49
+L GND #PWR037
 U 1 1 55A83EBF
 P 7775 4675
-F 0 "#PWR49" H 7775 4425 50  0001 C CNN
+F 0 "#PWR037" H 7775 4425 50  0001 C CNN
 F 1 "GND" H 7775 4525 50  0000 C CNN
 F 2 "" H 7775 4675 60  0000 C CNN
@@
 POWER
 $Comp
-L GND #PWR50
+L GND #PWR038
 U 1 1 55A83ED0
 P 7775 5350
-F 0 "#PWR50" H 7775 5100 50  0001 C CNN
+F 0 "#PWR038" H 7775 5100 50  0001 C CNN
 F 1 "GND" H 7775 5200 50  0000 C CNN
 F 2 "" H 7775 5350 60  0000 C CNN
@@
 POWER
 $Comp
-L GND #PWR46
+L GND #PWR039
 U 1 1 55A840A8
 P 6650 6050
-F 0 "#PWR46" H 6650 5800 50  0001 C CNN
+F 0 "#PWR039" H 6650 5800 50  0001 C CNN
 F 1 "GND" H 6650 5900 50  0000 C CNN
 F 2 "" H 6650 6050 60  0000 C CNN
@@
 POWER
 $Comp
-L GND #PWR51
+L GND #PWR040
 U 1 1 55A840CA
 P 7775 6050
-F 0 "#PWR51" H 7775 5800 50  0001 C CNN
+F 0 "#PWR040" H 7775 5800 50  0001 C CNN
 F 1 "GND" H 7775 5900 50  0000 C CNN
 F 2 "" H 7775 6050 60  0000 C CNN
@@
 POWER
 $Comp
-L GND #PWR55
+L GND #PWR041
 U 1 1 55A844A2
 P 8825 4675
-F 0 "#PWR55" H 8825 4425 50  0001 C CNN
+F 0 "#PWR041" H 8825 4425 50  0001 C CNN
 F 1 "GND" H 8825 4525 50  0000 C CNN
 F 2 "" H 8825 4675 60  0000 C CNN
@@
 POWER
 $Comp
-L GND #PWR56
+L GND #PWR042
 U 1 1 55A844B3
 P 8825 5350
-F 0 "#PWR56" H 8825 5100 50  0001 C CNN
+F 0 "#PWR042" H 8825 5100 50  0001 C CNN
 F 1 "GND" H 8825 5200 50  0000 C CNN
 F 2 "" H 8825 5350 60  0000 C CNN
@@
 POWER
 $Comp
-L GND #PWR57
+L GND #PWR043
 U 1 1 55A844E6
 P 8825 6050
-F 0 "#PWR57" H 8825 5800 50  0001 C CNN
+F 0 "#PWR043" H 8825 5800 50  0001 C CNN
 F 1 "GND" H 8825 5900 50  0000 C CNN
 F 2 "" H 8825 6050 60  0000 C CNN
@@
 $EndComp
 $Comp
-L GND #PWR60
+L GND #PWR044
 U 1 1 55A84508
 P 9950 6050
-F 0 "#PWR60" H 9950 5800 50  0001 C CNN
+F 0 "#PWR044" H 9950 5800 50  0001 C CNN
 F 1 "GND" H 9950 5900 50  0000 C CNN
 F 2 "" H 9950 6050 60  0000 C CNN
@@
 $EndComp
 $Comp
-L GND #PWR59
+L GND #PWR045
 U 1 1 55A844D5
 P 9950 5350
-F 0 "#PWR59" H 9950 5100 50  0001 C CNN
+F 0 "#PWR045" H 9950 5100 50  0001 C CNN
 F 1 "GND" H 9950 5200 50  0000 C CNN
 F 2 "" H 9950 5350 60  0000 C CNN
@@
 $EndComp
 $Comp
-L GND #PWR58
+L GND #PWR046
 U 1 1 55A844C4
 P 9950 4675
-F 0 "#PWR58" H 9950 4425 50  0001 C CNN
+F 0 "#PWR046" H 9950 4425 50  0001 C CNN
 F 1 "GND" H 9950 4525 50  0000 C CNN
 F 2 "" H 9950 4675 60  0000 C CNN
@@
 $EndComp
 $Comp
-L GND #PWR38
+L GND #PWR047
 U 1 1 55AABF17
 P 4825 1625
-F 0 "#PWR38" H 4825 1375 50  0001 C CNN
+F 0 "#PWR047" H 4825 1375 50  0001 C CNN
 F 1 "GND" H 4825 1475 50  0000 C CNN
 F 2 "" H 4825 1625 60  0000 C CNN
@@
 $EndComp
 $Comp
-L +3V3 #PWR37
+L +3V3 #PWR048
 U 1 1 55AABF5B
 P 4825 1425
-F 0 "#PWR37" H 4825 1275 50  0001 C CNN
+F 0 "#PWR048" H 4825 1275 50  0001 C CNN
 F 1 "+3V3" H 4825 1565 50  0000 C CNN
 F 2 "" H 4825 1425 60  0000 C CNN
@@
 NoConn ~ 6050 1925
 $Comp
-L +5V #PWR42
+L +5V #PWR049
 U 1 1 55AAC661
 P 6500 1225
-F 0 "#PWR42" H 6500 1075 50  0001 C CNN
+F 0 "#PWR049" H 6500 1075 50  0001 C CNN
 F 1 "+5V" H 6500 1365 50  0000 C CNN
 F 2 "" H 6500 1225 60  0000 C CNN
@@
 $EndComp
 $Comp
-L GND #PWR43
+L GND #PWR050
 U 1 1 55AAC741
 P 6500 1325
-F 0 "#PWR43" H 6500 1075 50  0001 C CNN
+F 0 "#PWR050" H 6500 1075 50  0001 C CNN
 F 1 "GND" H 6500 1175 50  0000 C CNN
 F 2 "" H 6500 1325 60  0000 C CNN
@@
 UART_EXT_RX
 $Comp
-L GND #PWR40
+L GND #PWR051
 U 1 1 55AD0E58
 P 5125 3300
-F 0 "#PWR40" H 5125 3050 50  0001 C CNN
+F 0 "#PWR051" H 5125 3050 50  0001 C CNN
 F 1 "GND" H 5125 3150 50  0000 C CNN
 F 2 "" H 5125 3300 60  0000 C CNN
@@
 I2C2_SCL
 $Comp
-L GND #PWR48
+L GND #PWR052
 U 1 1 55AD34BB
 P 6975 3275
-F 0 "#PWR48" H 6975 3025 50  0001 C CNN
+F 0 "#PWR052" H 6975 3025 50  0001 C CNN
 F 1 "GND" H 6975 3125 50  0000 C CNN
 F 2 "" H 6975 3275 60  0000 C CNN
@@
 $EndComp
 $Comp
-L +3.3V_A #PWR47
+L +3.3V_A #PWR053
 U 1 1 55AD362E
 P 6975 3125
-F 0 "#PWR47" H 6975 3085 30  0001 C CNN
+F 0 "#PWR053" H 6975 3085 30  0001 C CNN
 F 1 "+3.3V_A" H 6975 3235 30  0000 C CNN
 F 2 "" H 6975 3125 60  0000 C CNN
@@
 I2C1_SCL
 $Comp
-L GND #PWR53
+L GND #PWR054
 U 1 1 55B24BD4
 P 8200 3275
-F 0 "#PWR53" H 8200 3025 50  0001 C CNN
+F 0 "#PWR054" H 8200 3025 50  0001 C CNN
 F 1 "GND" H 8200 3125 50  0000 C CNN
 F 2 "" H 8200 3275 60  0000 C CNN
@@
 $EndComp
 $Comp
-L +3.3V_A #PWR52
+L +3.3V_A #PWR055
 U 1 1 55B24BDD
 P 8200 3125
-F 0 "#PWR52" H 8200 3085 30  0001 C CNN
+F 0 "#PWR055" H 8200 3085 30  0001 C CNN
 F 1 "+3.3V_A" H 8200 3235 30  0000 C CNN
 F 2 "" H 8200 3125 60  0000 C CNN
@@
 SPI1_CS1
 $Comp
-L +5V #PWR39
+L +5V #PWR056
 U 1 1 55B33C9C
 P 5125 3150
-F 0 "#PWR39" H 5125 3000 50  0001 C CNN
+F 0 "#PWR056" H 5125 3000 50  0001 C CNN
 F 1 "+5V" H 5125 3290 50  0000 C CNN
 F 2 "" H 5125 3150 60  0000 C CNN
@@
 $EndComp
 $Comp
-L +5V #PWR61
+L +5V #PWR057
 U 1 1 55B33EE7
 P 10200 3100
-F 0 "#PWR61" H 10200 2950 50  0001 C CNN
+F 0 "#PWR057" H 10200 2950 50  0001 C CNN
 F 1 "+5V" H 10200 3240 50  0000 C CNN
 F 2 "" H 10200 3100 60  0000 C CNN
@@
 $EndComp
 $Comp
-L GND #PWR62
+L GND #PWR058
 U 1 1 55B33F87
 P 10200 3250
-F 0 "#PWR62" H 10200 3000 50  0001 C CNN
+F 0 "#PWR058" H 10200 3000 50  0001 C CNN
 F 1 "GND" H 10200 3100 50  0000 C CNN
 F 2 "" H 10200 3250 60  0000 C CNN
@@
 $EndComp
 $Comp
-L GND #PWR54
+L GND #PWR059
 U 1 1 55B4173D
 P 8600 2250
-F 0 "#PWR54" H 8600 2000 50  0001 C CNN
+F 0 "#PWR059" H 8600 2000 50  0001 C CNN
 F 1 "GND" H 8600 2100 50  0000 C CNN
 F 2 "" H 8600 2250 60  0000 C CNN
@@
 $EndComp
 $Comp
-L GND #PWR63
+L GND #PWR060
 U 1 1 55B429BE
 P 10525 2250
-F 0 "#PWR63" H 10525 2000 50  0001 C CNN
+F 0 "#PWR060" H 10525 2000 50  0001 C CNN
 F 1 "GND" H 10525 2100 50  0000 C CNN
 F 2 "" H 10525 2250 60  0000 C CNN
@@
 POWER
 $Comp
-L GND #PWR41
+L GND #PWR061
 U 1 1 55B4F1B2
 P 5725 6225
-F 0 "#PWR41" H 5725 5975 50  0001 C CNN
+F 0 "#PWR061" H 5725 5975 50  0001 C CNN
 F 1 "GND" H 5725 6075 50  0000 C CNN
 F 2 "" H 5725 6225 60  0000 C CNN
@@
 Connection ~ 6125 1350
 $Comp
-L +3.3V_A #PWR29
+L +3.3V_A #PWR062
 U 1 1 55AE8E8A
 P 875 5500
-F 0 "#PWR29" H 875 5460 30  0001 C CNN
+F 0 "#PWR062" H 875 5460 30  0001 C CNN
 F 1 "+3.3V_A" H 875 5610 30  0000 C CNN
 F 2 "" H 875 5500 60  0000 C CNN
@@
 $EndComp
 $Comp
-L GND #PWR30
+L GND #PWR063
 U 1 1 55AE8F19
 P 875 5800
-F 0 "#PWR30" H 875 5550 50  0001 C CNN
+F 0 "#PWR063" H 875 5550 50  0001 C CNN
 F 1 "GND" H 875 5650 50  0000 C CNN
 F 2 "" H 875 5800 60  0000 C CNN
@@
 F 0 "CONN18" H 10600 4350 50  0000 C CNN
 F 1 "SPI" H 10600 3450 50  0000 C CNN
-F 2 "" H 10900 4200 39  0000 C CNN
+F 2 "_connectors:_Molex-PicoBlade-SMD-6" H 10900 4200 39  0001 C CNN
 F 3 "" H 10900 4200 39  0000 C CNN
 	1    11000 3650
@@
 F 0 "CONN19" H 8950 2175 59  0000 C CNN
 F 1 "ADC 3.3V" H 8950 1525 59  0000 C CNN
-F 2 "" H 8950 1600 59  0000 C CNN
+F 2 "_connectors:_Molex-PicoBlade-SMD-4" H 8950 1600 59  0001 C CNN
 F 3 "" H 8950 1600 59  0000 C CNN
 	1    8950 1600
@@
 F 0 "CONN20" H 10875 2175 59  0000 C CNN
 F 1 "ADC 5V" H 10875 1525 59  0000 C CNN
-F 2 "" H 10875 1600 59  0000 C CNN
+F 2 "_connectors:_Molex-PicoBlade-SMD-4" H 10875 1600 59  0001 C CNN
 F 3 "" H 10875 1600 59  0000 C CNN
 	1    10875 1600
